File: eagle/ESP8266 Programmer Board/Programmer Board v1.sch (EAGLE design)
At the start: 11 parts, among them J1 FTDI, J2 DCJ0202, U1 LM7833

Commit message: Updating switches
Parts:
- added D2: PROG, SparkFun-LED:LED3MM
- C1: value (none) -> 0.1uF
- C2: value (none) -> 10uF; device SparkFun-Capacitors:0.1UF-50V-20%(PTH)KIT-EZ -> SparkFun-Capacitors:10UF-25V-20%(PTH)KIT
- J1: device SparkFun-Connectors:ARDUINO_SERIAL_PROGRAMLONGPADS -> SparkFun-Connectors:FTDI_BASICPTH
- S2: value PROG -> (none); device SparkFun-Electromechanical:SWITCH-SPDTPTH -> SparkFun-Electromechanical:SWITCH-DPDTEG2211
Connections:
- removed net 3V3: JP1.7
- removed net CH_PD: JP1.3, S2.S
- removed net N$1: D1.C, R2.2
- new net N$3: D1.C, S2.4
- new net N$4: R2.2, S2.5
- net +3V3: now also C2.+, D2.A, JP1.3, JP1.7; no longer C2.1
- net GND: now also C2.-, J1.6, R2.1, S2.2; no longer C2.2, J1.GND, S2.P
- net GPIO0: now also S2.3
- net N$2: now also D2.C, S2.6; no longer R2.1, S2.O
- net RX: now also J1.3; no longer J1.TXO
- net TX: now also J1.2; no longer J1.RXI
Other:
- moved on the sheet: D1, J1, R2
Changed lines of the file:
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@@
 <setting verticaltext="up"/>
 </settings>
-<grid distance="0.1" unitdist="inch" unit="inch" style="dots" multiple="1" display="yes" altdistance="0.025" altunitdist="inch" altunit="inch"/>
+<grid distance="0.1" unitdist="inch" unit="inch" style="lines" multiple="1" display="no" altdistance="0.01" altunitdist="inch" altunit="inch"/>
 <layers>
 <layer number="1" name="Top" color="4" fill="1" visible="no" active="no"/>
@@
 <part name="JP1" library="adafruit" deviceset="PINHD-2X4" device="" value="ESP8266"/>
 <part name="R1" library="SparkFun-Resistors" deviceset="10KOHM-1/4W-1%(PTH)" device="HORIZ" value="10k"/>
-<part name="C1" library="SparkFun-Capacitors" deviceset="0.1UF-50V-20%(PTH)" device="KIT-EZ"/>
+<part name="C1" library="SparkFun-Capacitors" deviceset="0.1UF-50V-20%(PTH)" device="KIT-EZ" value="0.1uF"/>
 <part name="S1" library="SparkFun-Electromechanical" deviceset="SWITCH-MOMENTARY-2" device="PTH" value="RESET"/>
-<part name="S2" library="SparkFun-Electromechanical" deviceset="SWITCH-SPDT" device="PTH" value="PROG"/>
 <part name="U1" library="SparkFun-PowerIC" deviceset="V_REG_78XX" device="-TO-220" value="LM7833"/>
-<part name="J1" library="SparkFun-Connectors" deviceset="ARDUINO_SERIAL_PROGRAM" device="LONGPADS" value="FTDI"/>
+<part name="J1" library="SparkFun-Connectors" deviceset="FTDI_BASIC" device="PTH" value="FTDI"/>
 <part name="J2" library="con-jack" deviceset="DCJ0202" device=""/>
 <part name="+3V1" library="supply1" deviceset="+3V3" device=""/>
 <part name="GND1" library="supply1" deviceset="GND" device=""/>
 <part name="P+1" library="supply1" deviceset="VCC" device=""/>
-<part name="C2" library="SparkFun-Capacitors" deviceset="0.1UF-50V-20%(PTH)" device="KIT-EZ"/>
 <part name="GND2" library="supply1" deviceset="GND" device=""/>
 <part name="+3V2" library="supply1" deviceset="+3V3" device=""/>
-<part name="GND3" library="supply1" deviceset="GND" device=""/>
 <part name="GND4" library="supply1" deviceset="GND" device=""/>
 <part name="D1" library="SparkFun-LED" deviceset="LED" device="3MM" value="RUN"/>
 <part name="R2" library="SparkFun-Resistors" deviceset="10KOHM-1/4W-1%(PTH)" device="HORIZ" value="75"/>
 <part name="+3V3" library="supply1" deviceset="+3V3" device=""/>
+<part name="S2" library="SparkFun-Electromechanical" deviceset="SWITCH-DPDT" device="EG2211"/>
+<part name="D2" library="SparkFun-LED" deviceset="LED" device="3MM" value="PROG"/>
+<part name="GND3" library="supply1" deviceset="GND" device=""/>
+<part name="+3V4" library="supply1" deviceset="+3V3" device=""/>
+<part name="GND5" library="supply1" deviceset="GND" device=""/>
+<part name="C2" library="SparkFun-Capacitors" deviceset="10UF-25V-20%(PTH)" device="KIT" value="10uF"/>
 </parts>
 <sheets>
@@
 <instance part="C1" gate="G$1" x="5.08" y="83.82"/>
 <instance part="S1" gate="G$1" x="12.7" y="53.34"/>
-<instance part="S2" gate="1" x="38.1" y="58.42"/>
 <instance part="U1" gate="G$1" x="17.78" y="91.44"/>
 <instance part="J1" gate="G$1" x="76.2" y="81.28"/>
@@
 <instance part="GND1" gate="1" x="17.78" y="78.74"/>
 <instance part="P+1" gate="VCC" x="5.08" y="96.52"/>
-<instance part="C2" gate="G$1" x="33.02" y="83.82"/>
 <instance part="GND2" gate="1" x="5.08" y="48.26"/>
 <instance part="+3V2" gate="G$1" x="20.32" y="71.12"/>
-<instance part="GND3" gate="1" x="33.02" y="53.34"/>
 <instance part="GND4" gate="1" x="88.9" y="86.36"/>
-<instance part="D1" gate="G$1" x="45.72" y="78.74"/>
-<instance part="R2" gate="G$1" x="45.72" y="68.58" rot="R90"/>
-<instance part="+3V3" gate="G$1" x="45.72" y="86.36"/>
+<instance part="D1" gate="G$1" x="96.52" y="68.58"/>
+<instance part="R2" gate="G$1" x="127" y="53.34" rot="R90"/>
+<instance part="+3V3" gate="G$1" x="101.6" y="76.2"/>
+<instance part="S2" gate="G$1" x="114.3" y="53.34" rot="R180"/>
+<instance part="D2" gate="G$1" x="106.68" y="68.58"/>
+<instance part="GND3" gate="1" x="127" y="43.18"/>
+<instance part="+3V4" gate="G$1" x="50.8" y="63.5"/>
+<instance part="GND5" gate="1" x="91.44" y="58.42" rot="R90"/>
+<instance part="C2" gate="G$1" x="33.02" y="86.36"/>
 </instances>
 <busses>
@@
 </segment>
 <segment>
-<pinref part="J1" gate="G$1" pin="RXI"/>
+<pinref part="J1" gate="G$1" pin="2"/>
 <wire x1="81.28" y1="78.74" x2="86.36" y2="78.74" width="0.1524" layer="91"/>
 <label x="86.36" y="78.74" size="1.778" layer="95"/>
-</segment>
-</net>
-<net name="CH_PD" class="0">
-<segment>
-<pinref part="JP1" gate="A" pin="3"/>
-<wire x1="71.12" y1="55.88" x2="43.18" y2="55.88" width="0.1524" layer="91"/>
-<label x="55.88" y="55.88" size="1.778" layer="95"/>
-<pinref part="S2" gate="1" pin="S"/>
 </segment>
 </net>
@@
 </segment>
 </net>
-<net name="3V3" class="0">
-<segment>
-<pinref part="JP1" gate="A" pin="7"/>
-<wire x1="71.12" y1="50.8" x2="55.88" y2="50.8" width="0.1524" layer="91"/>
-<label x="55.88" y="50.8" size="1.778" layer="95"/>
-</segment>
-</net>
 <net name="GND" class="0">
 <segment>
@@
 <wire x1="78.74" y1="58.42" x2="88.9" y2="58.42" width="0.1524" layer="91"/>
 <label x="83.82" y="58.42" size="1.778" layer="95"/>
-</segment>
-<segment>
-<pinref part="C2" gate="G$1" pin="2"/>
+<pinref part="GND5" gate="1" pin="GND"/>
+</segment>
+<segment>
 <pinref part="GND1" gate="1" pin="GND"/>
 <wire x1="33.02" y1="81.28" x2="17.78" y2="81.28" width="0.1524" layer="91"/>
@@
 <wire x1="-5.08" y1="81.28" x2="5.08" y2="81.28" width="0.1524" layer="91"/>
 <junction x="5.08" y="81.28"/>
+<pinref part="C2" gate="G$1" pin="-"/>
 </segment>
 <segment>
@@
 </segment>
 <segment>
-<pinref part="GND3" gate="1" pin="GND"/>
-<wire x1="33.02" y1="55.88" x2="33.02" y2="58.42" width="0.1524" layer="91"/>
-<pinref part="S2" gate="1" pin="P"/>
-<wire x1="33.02" y1="58.42" x2="35.56" y2="58.42" width="0.1524" layer="91"/>
-</segment>
-<segment>
-<pinref part="J1" gate="G$1" pin="GND"/>
+<pinref part="J1" gate="G$1" pin="6"/>
 <wire x1="81.28" y1="88.9" x2="88.9" y2="88.9" width="0.1524" layer="91"/>
 <pinref part="GND4" gate="1" pin="GND"/>
+</segment>
+<segment>
+<pinref part="R2" gate="G$1" pin="1"/>
+<pinref part="GND3" gate="1" pin="GND"/>
+<wire x1="127" y1="48.26" x2="127" y2="45.72" width="0.1524" layer="91"/>
+<pinref part="S2" gate="G$1" pin="2"/>
+<wire x1="119.38" y1="50.8" x2="119.38" y2="45.72" width="0.1524" layer="91"/>
+<wire x1="119.38" y1="45.72" x2="127" y2="45.72" width="0.1524" layer="91"/>
+<junction x="127" y="45.72"/>
 </segment>
 </net>
@@
 <segment>
 <pinref part="JP1" gate="A" pin="6"/>
-<wire x1="78.74" y1="53.34" x2="88.9" y2="53.34" width="0.1524" layer="91"/>
 <label x="83.82" y="53.34" size="1.778" layer="95"/>
+<pinref part="S2" gate="G$1" pin="3"/>
+<wire x1="109.22" y1="53.34" x2="78.74" y2="53.34" width="0.1524" layer="91"/>
 </segment>
 </net>
@@
 </segment>
 <segment>
-<pinref part="J1" gate="G$1" pin="TXO"/>
+<pinref part="J1" gate="G$1" pin="3"/>
 <wire x1="81.28" y1="81.28" x2="86.36" y2="81.28" width="0.1524" layer="91"/>
 <label x="86.36" y="81.28" size="1.778" layer="95"/>
@@
 <wire x1="25.4" y1="91.44" x2="33.02" y2="91.44" width="0.1524" layer="91"/>
 <wire x1="33.02" y1="91.44" x2="33.02" y2="93.98" width="0.1524" layer="91"/>
-<pinref part="C2" gate="G$1" pin="1"/>
 <wire x1="33.02" y1="88.9" x2="33.02" y2="91.44" width="0.1524" layer="91"/>
 <junction x="33.02" y="91.44"/>
+<pinref part="C2" gate="G$1" pin="+"/>
 </segment>
 <segment>
@@
 </segment>
 <segment>
+<pinref part="D2" gate="G$1" pin="A"/>
 <pinref part="D1" gate="G$1" pin="A"/>
+<wire x1="106.68" y1="71.12" x2="101.6" y2="71.12" width="0.1524" layer="91"/>
 <pinref part="+3V3" gate="G$1" pin="+3V3"/>
-<wire x1="45.72" y1="81.28" x2="45.72" y2="83.82" width="0.1524" layer="91"/>
-</segment>
-</net>
-<net name="N$1" class="0">
-<segment>
+<wire x1="101.6" y1="71.12" x2="96.52" y2="71.12" width="0.1524" layer="91"/>
+<wire x1="101.6" y1="73.66" x2="101.6" y2="71.12" width="0.1524" layer="91"/>
+<junction x="101.6" y="71.12"/>
+</segment>
+<segment>
+<pinref part="JP1" gate="A" pin="7"/>
+<wire x1="71.12" y1="50.8" x2="50.8" y2="50.8" width="0.1524" layer="91"/>
+<label x="55.88" y="50.8" size="1.778" layer="95"/>
+<pinref part="+3V4" gate="G$1" pin="+3V3"/>
+<wire x1="50.8" y1="50.8" x2="50.8" y2="55.88" width="0.1524" layer="91"/>
+<pinref part="JP1" gate="A" pin="3"/>
+<wire x1="50.8" y1="55.88" x2="50.8" y2="60.96" width="0.1524" layer="91"/>
+<wire x1="71.12" y1="55.88" x2="50.8" y2="55.88" width="0.1524" layer="91"/>
+<label x="55.88" y="55.88" size="1.778" layer="95"/>
+<junction x="50.8" y="55.88"/>
+</segment>
+</net>
+<net name="N$2" class="0">
+<segment>
+<pinref part="S2" gate="G$1" pin="6"/>
+<pinref part="D2" gate="G$1" pin="C"/>
+<wire x1="109.22" y1="60.96" x2="106.68" y2="60.96" width="0.1524" layer="91"/>
+<wire x1="106.68" y1="60.96" x2="106.68" y2="63.5" width="0.1524" layer="91"/>
+</segment>
+</net>
+<net name="N$3" class="0">
+<segment>
+<pinref part="S2" gate="G$1" pin="4"/>
 <pinref part="D1" gate="G$1" pin="C"/>
+<wire x1="109.22" y1="55.88" x2="96.52" y2="55.88" width="0.1524" layer="91"/>
+<wire x1="96.52" y1="55.88" x2="96.52" y2="63.5" width="0.1524" layer="91"/>
+</segment>
+</net>
+<net name="N$4" class="0">
+<segment>
+<pinref part="S2" gate="G$1" pin="5"/>
 <pinref part="R2" gate="G$1" pin="2"/>
-</segment>
-</net>
-<net name="N$2" class="0">
-<segment>
-<pinref part="S2" gate="1" pin="O"/>
-<pinref part="R2" gate="G$1" pin="1"/>
-<wire x1="43.18" y1="60.96" x2="45.72" y2="60.96" width="0.1524" layer="91"/>
-<wire x1="45.72" y1="60.96" x2="45.72" y2="63.5" width="0.1524" layer="91"/>
-</segment>
-</net>
+<wire x1="119.38" y1="58.42" x2="127" y2="58.42" width="0.1524" layer="91"/>
+</segment>
+</net>

Commit message: Board routing
Parts:
- S2: device SparkFun-Electromechanical:SWITCH-DPDTEG2211 -> switch:A68-A31
Connections:
- net GND: now also S2A.P; no longer S2.2
- net GPIO0: now also S2A.S; no longer S2.3
- net N$2: now also S2B.S; no longer S2.6
- net N$3: now also S2B.O; no longer S2.4
- net N$4: now also S2B.P; no longer S2.5
Changed lines of the file:
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@@
 <part name="R2" library="SparkFun-Resistors" deviceset="10KOHM-1/4W-1%(PTH)" device="HORIZ" value="75"/>
 <part name="+3V3" library="supply1" deviceset="+3V3" device=""/>
-<part name="S2" library="SparkFun-Electromechanical" deviceset="SWITCH-DPDT" device="EG2211"/>
 <part name="D2" library="SparkFun-LED" deviceset="LED" device="3MM" value="PROG"/>
 <part name="GND3" library="supply1" deviceset="GND" device=""/>
@@
 <part name="GND5" library="supply1" deviceset="GND" device=""/>
 <part name="C2" library="SparkFun-Capacitors" deviceset="10UF-25V-20%(PTH)" device="KIT" value="10uF"/>
+<part name="S2" library="switch" deviceset="A68-A31" device=""/>
 </parts>
 <sheets>
@@
 <instance part="R2" gate="G$1" x="127" y="53.34" rot="R90"/>
 <instance part="+3V3" gate="G$1" x="101.6" y="76.2"/>
-<instance part="S2" gate="G$1" x="114.3" y="53.34" rot="R180"/>
 <instance part="D2" gate="G$1" x="106.68" y="68.58"/>
 <instance part="GND3" gate="1" x="127" y="43.18"/>
@@
 <instance part="GND5" gate="1" x="91.44" y="58.42" rot="R90"/>
 <instance part="C2" gate="G$1" x="33.02" y="86.36"/>
+<instance part="S2" gate="B" x="114.3" y="58.42" rot="R90"/>
+<instance part="S2" gate="A" x="114.3" y="48.26" rot="R90"/>
 </instances>
 <busses>
@@
 <pinref part="GND3" gate="1" pin="GND"/>
 <wire x1="127" y1="48.26" x2="127" y2="45.72" width="0.1524" layer="91"/>
-<pinref part="S2" gate="G$1" pin="2"/>
 <wire x1="119.38" y1="50.8" x2="119.38" y2="45.72" width="0.1524" layer="91"/>
 <wire x1="119.38" y1="45.72" x2="127" y2="45.72" width="0.1524" layer="91"/>
 <junction x="127" y="45.72"/>
+<pinref part="S2" gate="A" pin="P"/>
 </segment>
 </net>
@@
 <pinref part="JP1" gate="A" pin="6"/>
 <label x="83.82" y="53.34" size="1.778" layer="95"/>
-<pinref part="S2" gate="G$1" pin="3"/>
 <wire x1="109.22" y1="53.34" x2="78.74" y2="53.34" width="0.1524" layer="91"/>
+<pinref part="S2" gate="A" pin="S"/>
 </segment>
 </net>
@@
 <net name="N$2" class="0">
 <segment>
-<pinref part="S2" gate="G$1" pin="6"/>
 <pinref part="D2" gate="G$1" pin="C"/>
+<wire x1="106.68" y1="60.96" x2="106.68" y2="63.5" width="0.1524" layer="91"/>
+<pinref part="S2" gate="B" pin="S"/>
 <wire x1="109.22" y1="60.96" x2="106.68" y2="60.96" width="0.1524" layer="91"/>
-<wire x1="106.68" y1="60.96" x2="106.68" y2="63.5" width="0.1524" layer="91"/>
 </segment>
 </net>
 <net name="N$3" class="0">
 <segment>
-<pinref part="S2" gate="G$1" pin="4"/>
 <pinref part="D1" gate="G$1" pin="C"/>
+<wire x1="96.52" y1="55.88" x2="96.52" y2="63.5" width="0.1524" layer="91"/>
+<pinref part="S2" gate="B" pin="O"/>
 <wire x1="109.22" y1="55.88" x2="96.52" y2="55.88" width="0.1524" layer="91"/>
-<wire x1="96.52" y1="55.88" x2="96.52" y2="63.5" width="0.1524" layer="91"/>
 </segment>
 </net>
 <net name="N$4" class="0">
 <segment>
-<pinref part="S2" gate="G$1" pin="5"/>
 <pinref part="R2" gate="G$1" pin="2"/>
 <wire x1="119.38" y1="58.42" x2="127" y2="58.42" width="0.1524" layer="91"/>
-</segment>
-</net>
+<pinref part="S2" gate="B" pin="P"/>
+</segment>
+</net>
